File: kicad/photogate.kicad_sch (KiCad schematic)
At the start: 7 parts, among them J1 Output, Q1 SFH310, U1 74LS14

Commit message: doc changed
Parts:
- removed D1: LTE5208, symbol Device:LED
- removed J1: Output, symbol Connector:Conn_01x01_Pin
- removed Q1: SFH310, LED_THT:LED_D3.0mm_Clear, symbol Sensor_Optical:SFH309
- added J1: Conn_01x03_Pin, Connector_Wire:SolderWire-0.5sqmm_1x03_P4.6mm_D0.9mm_OD2.1mm, symbol Connector:Conn_01x03_Pin
- added J2: Conn_01x04_Pin, Connector_Wire:SolderWire-0.75sqmm_1x04_P4.8mm_D1.25mm_OD2.3mm, symbol Connector:Conn_01x04_Pin
- added unit 2 of U1
- R1, R3: footprint (none) -> Resistor_THT:R_Axial_DIN0207_L6.3mm_D2.5mm_P10.16mm_Horizontal
- R2: value > 47k -> 47k; footprint (none) -> Resistor_THT:R_Axial_DIN0207_L6.3mm_D2.5mm_P10.16mm_Horizontal
- U1: footprint (none) -> Package_DIP:DIP-14_W7.62mm_Socket
Connections:
- net GND: now also U1.7 (GND), J1.1 (Pin_1), J2.2 (Pin_2), J2.3 (Pin_3)
- net VCC: now also U1.14 (VCC), J1.3 (Pin_3)
- net at R2.2, U1.1: now also J2.1 (Pin_1)
- net at U1.2: now also J1.2 (Pin_2)
- net at R3.2, U1.11, U1.13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: now also U1.3; no longer U1.3
- net at R1.2: now also J2.4 (Pin_4)
Other:
- note added: "to the IR LED"
- note added: "to the phototransistor"
- moved on the sheet: R1, R2, R3
